File: piirilevy/robotti/robotti.kicad_pcb (KiCad board)
At the start: 2 copper layers, 86.7 x 68.6 mm, 64 parts, among them J1 VL53L1X, J2 VL53L1X, J3 XT30, J4 ST-LINK_V2, J5 UART, J6 Nema14, J7 Nema14, Q1 ALS-PT19-315C, SW1 SW_SPST, U1 SEN0373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

Commit message: PCB korjattu ei valmis
Parts:
- removed R7, R8: 10k, Resistor_SMD:R_0805_2012Metric
- moved R11 26.9 mm to (123.1, 91.0)
- moved R10 26.5 mm to (121.0, 91.0)
- moved R12 24.2 mm to (154.4, 76.7), turned to 270 degrees
- moved C24 22.3 mm to (120.0, 97.1)
- moved L1 21.6 mm to (138.5, 99.7), turned to 0 degrees
- moved C22 20.5 mm to (127.9, 91.2)
- moved R13 20.2 mm to (151.5, 76.7), turned to 270 degrees
- moved C23 17.3 mm to (132.0, 91.2), turned to 180 degrees
- moved R9 15.4 mm to (135.1, 90.3)
- moved U5 14.2 mm to (125.8, 96.2), turned to 180 degrees
- moved C25 12.9 mm to (138.5, 110.2)
- moved D4 7.11 mm to (127.0, 103.4), turned to 0 degrees
- moved C16 3.50 mm to (140.0, 62.3)
- moved C18 1.28 mm to (141.7, 60.1)
- moved C7 1.11 mm to (142.0, 65.0), turned to 180 degrees
Connections:
- C7 pad 1: VDD -> GND
- J1 pad 1: Net-(J1-Pad1) -> (no net)
- J1 pad 6: Net-(J1-Pad6) -> (no net)
- J1 pad 7: Net-(J1-Pad7) -> /PA9
- J2 pad 1: Net-(J2-Pad1) -> (no net)
- J2 pad 6: Net-(J2-Pad6) -> (no net)
- J2 pad 7: Net-(J2-Pad7) -> /PA8
- U1 pad 5: Net-(U1-Pad5) -> (no net)
- U2 pad 14: Net-(U2-Pad14) -> (no net)
- U2 pad 15: /PA1 -> (no net)
- U2 pad 16: /PA2 -> (no net)
- U2 pad 17: /PA3 -> (no net)
- U2 pad 4: Net-(U2-Pad4) -> (no net)
- U2 pad 40: /PC9 -> (no net)
- U2 pad 8: /PC0 -> (no net)
- U4 pad 1: Net-(U4-Pad1) -> (no net)
- U4 pad 10: Net-(U4-Pad10) -> (no net)
- U4 pad 11: Net-(U4-Pad11) -> (no net)
- U4 pad 16: Net-(U4-Pad16) -> (no net)
- U4 pad 17: Net-(U4-Pad17) -> (no net)
- U4 pad 18: Net-(U4-Pad18) -> (no net)
- U4 pad 7: Net-(U4-Pad7) -> (no net)
- U4 pad 8: Net-(U4-Pad8) -> (no net)
- U4 pad 9: Net-(U4-Pad9) -> (no net)
- U5 pad 2: Net-(U5-Pad2) -> (no net)
- U5 pad 6: Net-(U5-Pad6) -> (no net)
- U5 pad 9: Net-(U5-Pad9) -> GND
Routing:
- net VDD: track 396.8 -> 367.0 mm, vias 6 -> 4
- net VCC: track 89.4 -> 116.5 mm
- net Net-(D4-Pad2): track 20.1 -> 0.00 mm
- net /PA9: track 0.00 -> 15.3 mm
- net /PA8: track 0.00 -> 14.9 mm, vias 0 -> 2
- net Net-(C22-Pad2): track 7.47 -> 0.00 mm
- net Net-(R10-Pad2): track 6.17 -> 0.00 mm
- net Net-(J1-Pad6): track 5.03 -> 0.00 mm
- net Net-(J2-Pad6): track 3.06 -> 0.00 mm
- net /PC8: track 24.4 -> 26.9 mm
- net /PC1: track 29.5 -> 27.4 mm
- net /PC7: track 34.8 -> 35.3 mm
- net GND: vias 59 -> 46
- added copper zone on F.Cu, net Net-(C22-Pad2)
- added copper zone on F.Cu, net Net-(D4-Pad2)
- added copper zone on F.Cu, net Net-(R10-Pad2)
- added copper zone on F.Cu, net VCC
- added copper zone on F.Cu, net VDD

Commit message: PCB final tilattu ver.
Parts:
- U5: footprint Package_SO:HSOP-8-1EP_3.9x4.9mm_P1.27mm_EP2.41x3.1mm_ThermalVias -> robotti:HSOP-8-1EP_3.9x4.9mm_P1.27mm_EP2.41x3.1mm_ThermalVias
- moved C10 7.42 mm to (118.3, 83.3), turned to 270 degrees
- moved J3 5.05 mm to (155.5, 109.2), turned to 180 degrees
- moved C11 3.29 mm to (117.0, 76.3)
- moved C20 2.60 mm to (142.9, 72.9)
- moved R10 2.29 mm to (123.3, 91.0)
- moved C17 2.14 mm to (121.6, 73.9), turned to 270 degrees
- moved R11 2.10 mm to (121.0, 91.0)
- moved C15 2.03 mm to (140.5, 72.9)
- moved C12 2.03 mm to (106.1, 100.2), turned to 0 degrees
- moved C18 1.66 mm to (140.0, 60.2)
- moved C19 1.33 mm to (123.9, 73.9), turned to 90 degrees
- moved C7 1.33 mm to (143.2, 64.4)
- moved R9 1.26 mm to (136.0, 91.2), turned to 0 degrees
- moved C9 1.18 mm to (137.5, 77.2)
- moved C8 1.12 mm to (139.9, 77.2)
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Connections:
- J1 pad 1: (no net) -> Net-(J1-Pad1)
- J1 pad 6: (no net) -> Net-(J1-Pad6)
- J2 pad 1: (no net) -> Net-(J2-Pad1)
- J2 pad 6: (no net) -> Net-(J2-Pad6)
- J3 pad 1: VCC -> GND
- J3 pad 2: GND -> VCC
- U1 pad 5: (no net) -> Net-(U1-Pad5)
- U2 pad 14: (no net) -> Net-(U2-Pad14)
- U2 pad 15: (no net) -> /PA1
- U2 pad 16: (no net) -> /PA2
- U2 pad 17: (no net) -> /PA3
- U2 pad 4: (no net) -> Net-(U2-Pad4)
- U2 pad 40: (no net) -> /PC9
- U2 pad 8: (no net) -> /PC0
- U4 pad 1: (no net) -> Net-(U4-Pad1)
- U4 pad 10: (no net) -> Net-(U4-Pad10)
- U4 pad 11: (no net) -> Net-(U4-Pad11)
- U4 pad 16: (no net) -> Net-(U4-Pad16)
- U4 pad 17: (no net) -> Net-(U4-Pad17)
- U4 pad 18: (no net) -> Net-(U4-Pad18)
- U4 pad 7: (no net) -> Net-(U4-Pad7)
- U4 pad 8: (no net) -> Net-(U4-Pad8)
- U4 pad 9: (no net) -> Net-(U4-Pad9)
- U5 pad 2: (no net) -> Net-(U5-Pad2)
- U5 pad 6: (no net) -> Net-(U5-Pad6)
Routing:
- net VDD: track 367.0 -> 339.1 mm, vias 4 -> 6
- net /PC2: track 41.4 -> 30.9 mm, vias 0 -> 2
- net /PC3: track 43.6 -> 35.3 mm, vias 0 -> 2
- net /PB10: track 31.9 -> 37.7 mm
- net /PC1: track 27.4 -> 32.3 mm
- net /PB13: track 40.3 -> 45.2 mm
- net /PC8: track 26.9 -> 28.8 mm
- net /PA6: track 27.3 -> 29.1 mm
- net /PB12: track 22.4 -> 23.8 mm
- net Net-(C7-Pad2): track 3.87 -> 5.31 mm
- net VCC: track 116.5 -> 115.2 mm
- net /PA7: track 15.4 -> 16.7 mm
- net Net-(C5-Pad1): track 7.64 -> 6.56 mm
- net /PB8: track 39.1 -> 39.8 mm
- net /PC13: track 17.9 -> 18.7 mm
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Other:
- board size 86.7 x 68.6 mm -> 86.8 x 68.6 mm
- board text added: "Group 4 2021 Severi O. Valtteri A. Juha-Matti R."
