File: piirilevy/robotti/robotti.sch (KiCad schematic (older format))
At the start: 60 parts, among them J1 VL53L1X, J2 VL53L1X, J3 XT30, J4 ST-LINK_V2, J5 UART, J6 Nema14, J7 Nema14, Q1 ALS-PT19-315C, SW1 SW_SPST, U1 SEN0373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

Commit message: PCB korjattu ei valmis
Parts:
- removed R7, R8: 10k, Resistor_SMD:R_0805_2012Metric, symbol Device:R
Connections:
- net GND: now also C7.1, U5.9 (EP)
- net PA8: now also J2.7 (GPIO1)
- net PA9: now also J1.7 (GPIO1)
- net VDD: no longer C7.1
- no-connect marks 25 -> 22
Changed lines of the file:
@@
-	0    -1   -1   0
-$EndComp
-$Comp
-L power:VDD #PWR011
-U 1 1 606248D7
-P 4650 2700
-F 0 "#PWR011" H 4650 2550 50  0001 C CNN
-F 1 "VDD" V 4665 2827 50  0000 L CNN
-F 2 "" H 4650 2700 50  0001 C CNN
-F 3 "" H 4650 2700 50  0001 C CNN
-	1    4650 2700
 	0    -1   -1   0
 $EndComp
@@
 	0    -1   -1   0
 $EndComp
-$Comp
-L Device:R R7
-U 1 1 6066EC43
-P 7800 4150
-F 0 "R7" V 7600 4150 50  0000 C CNN
-F 1 "10k" V 7700 4150 50  0000 C CNN
-F 2 "Resistor_SMD:R_0805_2012Metric" V 7730 4150 50  0001 C CNN
-F 3 "~" H 7800 4150 50  0001 C CNN
-	1    7800 4150
-	0    1    1    0
-$EndComp
 Text Label 6700 4700 2    50   ~ 0
 PB7
@@
 PB6
 Wire Wire Line
-	8100 4650 7600 4650
-Wire Wire Line
 	7950 4550 8100 4550
-Wire Wire Line
-	8000 4250 8100 4250
 $Comp
 L power:GND #PWR020
@@
 	0    -1   -1   0
 $EndComp
-$Comp
-L Device:R R8
-U 1 1 6067BCAC
-P 7800 5050
-F 0 "R8" V 7600 5050 50  0000 C CNN
-F 1 "10k" V 7700 5050 50  0000 C CNN
-F 2 "Resistor_SMD:R_0805_2012Metric" V 7730 5050 50  0001 C CNN
-F 3 "~" H 7800 5050 50  0001 C CNN
-	1    7800 5050
-	0    1    1    0
-$EndComp
-Wire Wire Line
-	8100 5550 7600 5550
 Wire Wire Line
 	7950 5450 8100 5450
-Wire Wire Line
-	8000 5150 8100 5150
 Wire Wire Line
 	8100 4450 7100 4450
@@
 $EndComp
 Wire Wire Line
-	1900 6950 1900 7400
+	1900 6950 1900 7100
 Wire Wire Line
 	1900 7400 2100 7400
@@
 Wire Wire Line
 	3150 1350 3200 1350
-NoConn ~ 2000 6950
 NoConn ~ 2400 6750
 NoConn ~ 1400 6550
@@
 NoConn ~ 9200 1900
 NoConn ~ 8100 4750
-NoConn ~ 8100 4150
-NoConn ~ 8100 5050
 NoConn ~ 8100 5650
 Text Label 6050 1900 1    50   ~ 0
@@
 Text Label 7650 5350 0    50   ~ 0
 SDA_VL53_2
-Wire Wire Line
-	8000 5150 8000 5050
-Wire Wire Line
-	7600 5050 7600 5550
-Connection ~ 7600 5550
-Wire Wire Line
-	8000 4150 7950 4150
-Wire Wire Line
-	8000 4150 8000 4250
-Wire Wire Line
-	7600 4150 7600 4650
-Connection ~ 7600 4650
 Text Label 7650 4350 0    50   ~ 0
 SCL_VL53_1
@@
 NoConn ~ 6700 2500
 NoConn ~ 6700 2600
-NoConn ~ 6700 3100
-NoConn ~ 6700 3200
 NoConn ~ 4850 4000
 NoConn ~ 4800 4900
@@
 NoConn ~ 1650 1750
 Wire Wire Line
-	7600 4150 7650 4150
-Wire Wire Line
-	7950 5050 8000 5050
-Wire Wire Line
-	7650 5050 7600 5050
-Wire Wire Line
-	7550 4650 7600 4650
-Wire Wire Line
-	7550 5550 7600 5550
-Wire Wire Line
 	7050 2150 7100 2150
 Wire Wire Line
@@
 Wire Wire Line
 	6700 1200 7550 1200
+Wire Wire Line
+	7550 4650 8100 4650
+Wire Wire Line
+	7550 5550 8100 5550
+NoConn ~ 8100 4250
+NoConn ~ 8100 5150
+Wire Wire Line
+	8100 4150 7850 4150
+Wire Wire Line
+	8100 5050 7850 5050
+Text Label 7850 4150 0    50   ~ 0
+PA9
+Text Label 7850 5050 0    50   ~ 0
+PA8
+Wire Wire Line
+	2000 6950 2000 7100
+Wire Wire Line
+	2000 7100 1900 7100
+Connection ~ 1900 7100
+Wire Wire Line
+	1900 7100 1900 7400
+Wire Wire Line
+	4600 2500 4600 2700
+Wire Wire Line
+	4600 2700 4650 2700
 $EndSCHEMATC

Commit message: PCB final tilattu ver.
Parts:
- U5: footprint Package_SO:HSOP-8-1EP_3.9x4.9mm_P1.27mm_EP2.41x3.1mm_ThermalVias -> robotti:HSOP-8-1EP_3.9x4.9mm_P1.27mm_EP2.41x3.1mm_ThermalVias
Connections:
- net GND: now also J3.1 (GND); no longer J3.2 (VCC)
- net VCC: now also J3.2 (VCC); no longer J3.1 (GND)
Other:
- moved on the sheet: J3
Changed lines of the file:
@@
 F 0 "U5" H 2150 7050 50  0000 C CNN
 F 1 "L5973D" H 2150 6950 50  0000 C CNN
-F 2 "Package_SO:HSOP-8-1EP_3.9x4.9mm_P1.27mm_EP2.41x3.1mm_ThermalVias" H 2050 6200 50  0001 L CNN
+F 2 "robotti:HSOP-8-1EP_3.9x4.9mm_P1.27mm_EP2.41x3.1mm_ThermalVias" H 2050 6200 50  0001 L CNN
 F 3 "http://www.st.com/resource/en/datasheet/l5973d.pdf" H 1900 6650 50  0001 C CNN
 	1    1900 6650
@@
 $EndComp
 $Comp
-L robotti_library:XT30 J3
-U 1 1 607FB2C4
-P 1900 5450
-F 0 "J3" V 1891 5292 50  0000 R CNN
-F 1 "XT30" V 1982 5292 50  0000 R CNN
-F 2 "Connector_AMASS:AMASS_XT30U-F_1x02_P5.0mm_Vertical" H 1900 5450 50  0001 C CNN
-F 3 "~" H 1900 5450 50  0001 C CNN
-	1    1900 5450
-	0    -1   1    0
-$EndComp
-$Comp
 L power:GND #PWR028
 U 1 1 6081506E
-P 2000 5650
-F 0 "#PWR028" H 2000 5400 50  0001 C CNN
-F 1 "GND" V 2005 5522 50  0000 R CNN
-F 2 "" H 2000 5650 50  0001 C CNN
-F 3 "" H 2000 5650 50  0001 C CNN
-	1    2000 5650
+P 1800 5650
+F 0 "#PWR028" H 1800 5400 50  0001 C CNN
+F 1 "GND" V 1805 5522 50  0000 R CNN
+F 2 "" H 1800 5650 50  0001 C CNN
+F 3 "" H 1800 5650 50  0001 C CNN
+	1    1800 5650
 	1    0    0    -1
 $EndComp
@@
 Wire Wire Line
 	750  7400 1050 7400
-Wire Wire Line
-	1900 5650 1900 6200
 $Comp
 L power:GND #PWR027
@@
 Wire Wire Line
 	1750 6200 1900 6200
-Connection ~ 1900 6200
 Wire Wire Line
 	1900 6200 1900 6350
@@
 L power:VCC #PWR039
 U 1 1 606DF10C
-P 1650 5650
-F 0 "#PWR039" H 1650 5500 50  0001 C CNN
-F 1 "VCC" V 1665 5777 50  0000 L CNN
-F 2 "" H 1650 5650 50  0001 C CNN
-F 3 "" H 1650 5650 50  0001 C CNN
-	1    1650 5650
-	0    -1   -1   0
-$EndComp
-Wire Wire Line
-	1650 5650 1900 5650
-Connection ~ 1900 5650
+P 2000 5750
+F 0 "#PWR039" H 2000 5600 50  0001 C CNN
+F 1 "VCC" V 2015 5877 50  0000 L CNN
+F 2 "" H 2000 5750 50  0001 C CNN
+F 3 "" H 2000 5750 50  0001 C CNN
+	1    2000 5750
+	0    1    1    0
+$EndComp
 $Comp
 L power:VCC #PWR040
@@
 Wire Wire Line
 	4600 2700 4650 2700
+$Comp
+L robotti_library:XT30 J3
+U 1 1 607FB2C4
+P 1800 5450
+F 0 "J3" V 1791 5292 50  0000 R CNN
+F 1 "XT30" V 1882 5292 50  0000 R CNN
+F 2 "Connector_AMASS:AMASS_XT30U-F_1x02_P5.0mm_Vertical" H 1800 5450 50  0001 C CNN
+F 3 "~" H 1800 5450 50  0001 C CNN
+	1    1800 5450
+	0    -1   1    0
+$EndComp
+Wire Wire Line
+	1900 5650 1900 5750
+Connection ~ 1900 6200
+Wire Wire Line
+	2000 5750 1900 5750
+Connection ~ 1900 5750
+Wire Wire Line
+	1900 5750 1900 6200
 $EndSCHEMATC
